Commit message: attempt laser sensor addition

File: workspace/limo_simulation/urdf/limo_four_diff.xacro (robot description, xacro)
@@ -64,3 +64,6 @@
         <origin xyz="${-wheelbase/2} ${-track/2} ${wheel_vertical_offset}" rpy="${M_PI} 0 0" />
     </xacro:limo_wheel>
+    <xacro:limo_laser parent_prefix="base_link" frame_prefix="laser">
+        <origin xyz="0.05 0 0.2" rpy="0 0 0"/>
+    </xacro:limo_laser>
 </robot>

File: workspace/limo_simulation/urdf/limo_xacro.xacro (robot description, xacro)
@@ -63,4 +63,26 @@
                 </geometry>
             </collision>
+            <sensor name="lidar" type="ray">
+                <pose>0 0 0.1 0 0 0</pose>
+                <update_rate>30</update_rate>
+                <ray>
+                    <scan>
+                        <horizontal>
+                            <samples>720</samples>
+                            <resolution>1</resolution>
+                            <min_angle>-1.57</min_angle>
+                            <max_angle>1.57</max_angle>
+                        </horizontal>
+                    </scan>
+                    <range>
+                        <min>0.1</min>
+                        <max>10.0</max>
+                    </range>
+                </ray>
+                <plugin name="ros_gz_lidar_bridge" filename="gz-ros2-laser-sensor-system">
+                    <topic>/scan</topic>
+                    <frame_id>laser_link</frame_id>
+                </plugin>
+            </sensor>
         </link>
         <joint type="fixed" name="laser_joint">
